File: rp2040.kicad_sch (KiCad schematic)
At the start: 25 parts, among them J10 Conn_01x02, J11 Conn_01x06, U5 W25Q32JVSS, U6 RP2040, Y1 12.0MHz

Commit message: Add waferspace Main PCB
Signed-off-by: Leo Moser <leomoser99@gmail.com>
Parts:
- C31, C33, C34, C35, C36, C38, C39, C40, C41: LCSC C100072 -> C1525
- C32, C37: LCSC C5673 -> C15849
- R34, R35, R36, R38, R39, R40: LCSC C471764 -> C25744
- R37: LCSC C202394 -> C11702
- U5: LCSC C82344 -> C179173
